Commit message: higher table

File: allegro_kuka_description/models/table.urdf.xacro (robot description, xacro)
@@ -13,5 +13,6 @@
        xmlns:controller="http://playerstage.sourceforge.net/gazebo/xmlschema/#controller"
        xmlns:physics="http://playerstage.sourceforge.net/gazebo/xmlschema/#physics">
-  <property name="table_height" value="0.13" />
+  <!-- <property name="table_height" value="0.13" /> -->
+  <property name="table_height" value="0.33" />
   <property name="table_width"  value="0.4" />
   <property name="table_depth"  value="0.4" />
@@ -25,5 +26,5 @@
   <property name="M_PI" value="3.1415926535897931" />
 <joint name="world_joint3"  type="fixed">
-    <origin xyz="0.8 -0.0 0.03" rpy="0 0 0" />
+    <origin xyz="-0.8 -0.0 0.03" rpy="0 0 0" />
     <parent link="world"/>
     <child link="table_top_link"/>
@@ -56,6 +57,8 @@
   <gazebo reference="table_top_link">
     <material>Gazebo/LightWood</material>
-    <mu1>50.0</mu1>
-    <mu2>50.0</mu2>
+    <!-- <mu1>50.0</mu1> -->
+    <!-- <mu2>50.0</mu2> -->
+    <mu1>0.0</mu1>
+    <mu2>0.0</mu2>
     <kp>1000000.0</kp>
     <kd>1.0</kd>
