Commit message: added/modified hand/robot models for RAS2016 paper revision

File: allegro_kuka_description/models/allegro_hand_on_kuka_axischanged.urdf.xacro (robot description, xacro)
@@ -4,5 +4,5 @@
     <xacro:include filename="$(find lwr_description)/model/materials.xml"/>
     <xacro:include filename="$(find allegro_hand_description_nico)/models/common.urdf.xacro"/>
-    <xacro:include filename="$(find allegro_hand_description_nico)/models/hand.urdf.xacro"/>
+    <xacro:include filename="$(find allegro_hand_description_nico)/models/hand_axischanged.urdf.xacro"/>
     <!-- This plugin outputs the robot's joint positions and inputs joint torques -->
     <gazebo>
@@ -24,13 +24,7 @@
             <update_rate>20</update_rate>
             <bumperTopicName>/link_collision_sensor</bumperTopicName>
+            <frameName/>
         </plugin>
     </gazebo>
-<!--         <gazebo>
-        <plugin filename="libgazebo_ros_my_world_manager_plugin.so" name="world_manager">
-            <always_on>true</always_on>
-            <update_rate>20</update_rate>
-            <bumperTopicName>/link_collision_sensor</bumperTopicName>
-        </plugin>
-    </gazebo> -->
     <!-- Kuka -->
     <kuka_lwr_arm name="lwr" parent="aluplate" right="1" tool_name="">

File: allegro_kuka_description/models/allegro_hand_released_limits_on_kuka.urdf.xacro (robot description, xacro)
@@ -4,5 +4,5 @@
     <xacro:include filename="$(find lwr_description)/model/materials.xml"/>
     <xacro:include filename="$(find allegro_hand_description_nico)/models/common.urdf.xacro"/>
-    <xacro:include filename="$(find allegro_hand_description_nico)/models/hand.urdf.xacro"/>
+    <xacro:include filename="$(find allegro_hand_description_nico)/models/hand_released_limits.urdf.xacro"/>
     <!-- This plugin outputs the robot's joint positions and inputs joint torques -->
     <gazebo>
@@ -24,13 +24,7 @@
             <update_rate>20</update_rate>
             <bumperTopicName>/link_collision_sensor</bumperTopicName>
+            <frameName/>
         </plugin>
     </gazebo>
-<!--         <gazebo>
-        <plugin filename="libgazebo_ros_my_world_manager_plugin.so" name="world_manager">
-            <always_on>true</always_on>
-            <update_rate>20</update_rate>
-            <bumperTopicName>/link_collision_sensor</bumperTopicName>
-        </plugin>
-    </gazebo> -->
     <!-- Kuka -->
     <kuka_lwr_arm name="lwr" parent="aluplate" right="1" tool_name="">

File: allegro_kuka_description/models/allegro_hand_released_limits_on_kuka_axischanged.urdf.xacro (robot description, xacro)
@@ -4,5 +4,6 @@
     <xacro:include filename="$(find lwr_description)/model/materials.xml"/>
     <xacro:include filename="$(find allegro_hand_description_nico)/models/common.urdf.xacro"/>
-    <xacro:include filename="$(find allegro_hand_description_nico)/models/hand.urdf.xacro"/>
+    <!-- <xacro:include filename="$(find allegro_hand_description_nico)/models/hand_released_limits.urdf.xacro"/> -->
+    <xacro:include filename="$(find allegro_hand_description_nico)/models/hand_released_limits_axischanged.urdf.xacro"/>
     <!-- This plugin outputs the robot's joint positions and inputs joint torques -->
     <gazebo>
@@ -24,13 +25,7 @@
             <update_rate>20</update_rate>
             <bumperTopicName>/link_collision_sensor</bumperTopicName>
+            <frameName/>
         </plugin>
     </gazebo>
-<!--         <gazebo>
-        <plugin filename="libgazebo_ros_my_world_manager_plugin.so" name="world_manager">
-            <always_on>true</always_on>
-            <update_rate>20</update_rate>
-            <bumperTopicName>/link_collision_sensor</bumperTopicName>
-        </plugin>
-    </gazebo> -->
     <!-- Kuka -->
     <kuka_lwr_arm name="lwr" parent="aluplate" right="1" tool_name="">

File: allegro_kuka_description/models/sh_hand_on_kuka.urdf.xacro (robot description, xacro)
@@ -4,7 +4,11 @@
     <xacro:include filename="$(find lwr_description)/model/materials.xml"/>
     <xacro:include filename="$(find allegro_hand_description_nico)/models/common.urdf.xacro"/>
-    <xacro:include filename="$(find allegro_hand_description_nico)/models/hand.urdf.xacro"/>
-    <!-- This plugin outputs the robot's joint positions and inputs joint torques -->
-    <gazebo>
+    <!-- <xacro:include filename="$(find allegro_hand_description_nico)/models/hand.urdf.xacro"/> -->
+    <!-- <xacro:include filename="$(find sr_description)/materials.urdf.xacro" /> -->
+    <xacro:include filename="$(find sr_description)/hand/xacro/full_hand.urdf.xacro" />
+    <xacro:include filename="$(find sr_description)/other/xacro/gazebo/gazebo.urdf.xacro" />
+    <!-- hand with cylindrical base drifts in gazebo, attach it to the world -->
+      <!-- This plugin outputs the robot's joint positions and inputs joint torques -->
+      <gazebo>
         <plugin filename="libmy_robot_plugin.so" name="input_all_torques">
             <topicName>/lwr/input_torques/ </topicName>
@@ -13,9 +17,9 @@
     </gazebo>
     <!-- Sets a joint position (for replay)  -->
-    <gazebo>
+<!--     <gazebo>
         <plugin filename="libset_joint_position_plugin.so" name="set_joint_position">
             <topicName>/set_gazebo_joint_states </topicName>
         </plugin>
-    </gazebo>
+    </gazebo> -->
     <!-- Streams the contacts  -->
     <gazebo>
@@ -24,13 +28,7 @@
             <update_rate>20</update_rate>
             <bumperTopicName>/link_collision_sensor</bumperTopicName>
+            <frameName/>
         </plugin>
     </gazebo>
-<!--         <gazebo>
-        <plugin filename="libgazebo_ros_my_world_manager_plugin.so" name="world_manager">
-            <always_on>true</always_on>
-            <update_rate>20</update_rate>
-            <bumperTopicName>/link_collision_sensor</bumperTopicName>
-        </plugin>
-    </gazebo> -->
     <!-- Kuka -->
     <kuka_lwr_arm name="lwr" parent="aluplate" right="1" tool_name="">
@@ -62,4 +60,17 @@
     <link name="world"/>
     <!-- Hand -->
-    <xacro:ahand left="-1" parent_link="lwr_arm_7_link" prefix="ahand" rpy="0 0 0" xyz="0 0 0.1"/>
-</robot>
+    <!-- <xacro:ahand left="-1" parent_link="lwr_arm_7_link" prefix="ahand" rpy="0 0 0" xyz="0 0 0.1"/> -->
+<!--
+  <joint name="lh_world_joint" type="fixed">
+    <parent link="world" />
+    <child link="lh_forearm" />
+    <origin xyz="0.0 0.0 0.0" rpy="0.0 0.0 0.0" />
+  </joint> -->
+    <xacro:shadowhand muscletrans="false" muscle="false" bio="false" bt_sp="false"
+      ubi="false" eli="false" reflect="-1.0" prefix="lh_" lf="true" />
+    <joint name="lh_world_joint" type="fixed">
+        <parent link="lwr_arm_7_link" />
+        <child link="lh_forearm" />
+        <origin xyz="0.0 0.0 0.0" rpy="0.0 0.0 0.0" />
+    </joint>
+  </robot>
