Commit message: synced my two robots with 2 variats of allegrohand

File: allegro_kuka_description/models/allegro_hand_on_kuka.urdf.xacro (robot description, xacro)
@@ -1,4 +1,3 @@
-<robot name="LWR"
-    xmlns:xacro="http://www.ros.org/wiki/xacro">
+<robot name="LWR" xmlns:xacro="http://www.ros.org/wiki/xacro">
     <!-- Some macros used by the urdf -->
     <xacro:include filename="$(find lwr_description)/model/kuka_lwr_arm.urdf.xacro"/>
@@ -6,58 +5,55 @@
     <xacro:include filename="$(find allegro_hand_description_nico)/models/common.urdf.xacro"/>
     <xacro:include filename="$(find allegro_hand_description_nico)/models/hand.urdf.xacro"/>
-    <!-- Creates controllers for the arm, unused -->
     <!-- This plugin outputs the robot's joint positions and inputs joint torques -->
     <gazebo>
-        <plugin name="input_all_torques" filename="libmy_robot_plugin.so">
-            <topicName> /lwr/input_torques/ </topicName>
-            <bodyName> lwr_arm_7_link </bodyName>
+        <plugin filename="libmy_robot_plugin.so" name="input_all_torques">
+            <topicName>/lwr/input_torques/ </topicName>
+            <bodyName>lwr_arm_7_link </bodyName>
         </plugin>
     </gazebo>
+    <!-- Sets a joint position (for replay)  -->
     <gazebo>
-        <plugin name="set_joint_position" filename="libset_joint_position_plugin.so">
-            <topicName> /set_gazebo_joint_states </topicName>
+        <plugin filename="libset_joint_position_plugin.so" name="set_joint_position">
+            <topicName>/set_gazebo_joint_states </topicName>
         </plugin>
     </gazebo>
     <!-- Streams the contacts  -->
     <gazebo>
-      <plugin name="link_collision_sensor" filename="libgazebo_ros_my_contact_plugin.so">
-       <always_on>true</always_on>
-       <update_rate>20</update_rate>
-       <bumperTopicName>/link_collision_sensor</bumperTopicName>
-       <frameName></frameName>
-   </plugin>
-</gazebo>
-<!-- Kuka -->
-<kuka_lwr_arm parent="aluplate" name="lwr" right="1" tool_name="">
-    <origin xyz="0 0 0" rpy="0 0 0"/>
-</kuka_lwr_arm>
-<!-- AluPlate -->
-<joint name="world_joint2"  type="fixed">
-    <origin xyz="0 0 0.03" rpy="0 0 0" />
-    <parent link="world"/>
-    <child link="aluplate"/>
-</joint>
-<link name="aluplate">
-    <visual>
-        <origin xyz="0 0 0.01" />
-        <geometry>
-            <box size="0.2 0.2 0.02" xyz="0.0 0.0 0.0"/>
-        </geometry>
-        <material name="Silver" />
-    </visual>
-    <collision name ='aluplate_collision'>
-        <geometry>
-         <box size="0.2 0.2 0.02" xyz="0.0 0.0 0.0"/>
-     </geometry>
- </collision>
-</link>
-<gazebo reference="aluplate">
-    <material value="Gazebo/Grey"/>
-</gazebo>
-<link name="world"/>
-<!-- Hand -->
-<xacro:ahand
-   prefix="ahand"
-   parent_link="lwr_arm_7_link"
-   xyz="0 0 0.1" rpy="0 0 0" left="-1"/>
+        <plugin filename="libgazebo_ros_my_contact_plugin.so" name="link_collision_sensor">
+            <always_on>true</always_on>
+            <update_rate>20</update_rate>
+            <bumperTopicName>/link_collision_sensor</bumperTopicName>
+            <frameName/>
+        </plugin>
+    </gazebo>
+    <!-- Kuka -->
+    <kuka_lwr_arm name="lwr" parent="aluplate" right="1" tool_name="">
+        <origin rpy="0 0 0" xyz="0 0 0"/>
+    </kuka_lwr_arm>
+    <!-- AluPlate -->
+    <joint name="world_joint2" type="fixed">
+        <origin rpy="0 0 0" xyz="0.0 0.0 0.03"/>
+        <parent link="world"/>
+        <child link="aluplate"/>
+    </joint>
+    <link name="aluplate">
+        <visual>
+            <origin xyz="0 0 0.01"/>
+            <geometry>
+                <box size="0.2 0.2 0.02" xyz="0.0 0.0 0.0"/>
+            </geometry>
+            <material name="Silver"/>
+        </visual>
+        <collision name="aluplate_collision">
+            <geometry>
+                <box size="0.2 0.2 0.02" xyz="0.0 0.0 0.0"/>
+            </geometry>
+        </collision>
+    </link>
+    <gazebo reference="aluplate">
+        <material value="Gazebo/Grey"/>
+    </gazebo>
+    <link name="world"/>
+    <!-- Hand -->
+    <xacro:ahand left="-1" parent_link="lwr_arm_7_link" prefix="ahand" rpy="0 0 0" xyz="0 0 0.1"/>
 </robot>

File: allegro_kuka_description/models/allegro_hand_on_kuka_stl_mesh_hand.urdf.xacro (robot description, xacro)
@@ -1,59 +1,59 @@
-<robot name="LWR"
-    xmlns:xacro="http://www.ros.org/wiki/xacro">
+<robot name="LWR" xmlns:xacro="http://www.ros.org/wiki/xacro">
     <!-- Some macros used by the urdf -->
     <xacro:include filename="$(find lwr_description)/model/kuka_lwr_arm.urdf.xacro"/>
     <xacro:include filename="$(find lwr_description)/model/materials.xml"/>
     <xacro:include filename="$(find allegro_hand_description_nico)/models/common.urdf.xacro"/>
-    <!-- <xacro:include filename="$(find allegro_hand_description_nico)/models/hand.urdf.xacro"/> -->
     <xacro:include filename="$(find allegro_hand_description_nico)/models/hand_new_mesh.urdf.xacro"/>
-    <!-- Creates controllers for the arm, unused -->
     <!-- This plugin outputs the robot's joint positions and inputs joint torques -->
     <gazebo>
-        <plugin name="input_all_torques" filename="libmy_robot_plugin.so">
-            <topicName> /lwr/input_torques/ </topicName>
-            <bodyName> lwr_arm_7_link </bodyName>
+        <plugin filename="libmy_robot_plugin.so" name="input_all_torques">
+            <topicName>/lwr/input_torques/ </topicName>
+            <bodyName>lwr_arm_7_link </bodyName>
+        </plugin>
+    </gazebo>
+    <!-- Sets a joint position (for replay)  -->
+    <gazebo>
+        <plugin filename="libset_joint_position_plugin.so" name="set_joint_position">
+            <topicName>/set_gazebo_joint_states </topicName>
         </plugin>
     </gazebo>
     <!-- Streams the contacts  -->
     <gazebo>
-      <plugin name="link_collision_sensor" filename="libgazebo_ros_my_contact_plugin.so">
-         <always_on>true</always_on>
-         <update_rate>20</update_rate>
-         <bumperTopicName>/link_collision_sensor</bumperTopicName>
-         <frameName></frameName>
-     </plugin>
+        <plugin filename="libgazebo_ros_my_contact_plugin.so" name="link_collision_sensor">
+            <always_on>true</always_on>
+            <update_rate>20</update_rate>
+            <bumperTopicName>/link_collision_sensor</bumperTopicName>
+            <frameName/>
+        </plugin>
     </gazebo>
-<!-- Kuka -->
- <kuka_lwr_arm parent="aluplate" name="lwr" right="1" tool_name="">
-    <origin xyz="0 0 0" rpy="0 0 0"/>
-</kuka_lwr_arm>
-<!-- AluPlate -->
-<joint name="world_joint2"  type="fixed">
-    <origin xyz="0 0 0.03" rpy="0 0 0" />
-    <parent link="world"/>
-    <child link="aluplate"/>
-</joint>
-<link name="aluplate">
-    <visual>
-        <origin xyz="0 0 0.01" />
-        <geometry>
-            <box size="0.2 0.2 0.02" xyz="0.0 0.0 0.0"/>
-        </geometry>
-        <material name="Silver" />
-    </visual>
-    <collision name ='aluplate_collision'>
-        <geometry>
-           <box size="0.2 0.2 0.02" xyz="0.0 0.0 0.0"/>
-       </geometry>
-   </collision>
-</link>
-<gazebo reference="aluplate">
-    <material value="Gazebo/Grey"/>
-</gazebo>
-<link name="world"/>
-<!-- Hand -->
-<xacro:ahand
- prefix="ahand"
- parent_link="lwr_arm_7_link"
- xyz="0 0 0.1" rpy="0 0 0" left="-1"/>
+    <!-- Kuka -->
+    <kuka_lwr_arm name="lwr" parent="aluplate" right="1" tool_name="">
+        <origin rpy="0 0 0" xyz="0 0 0"/>
+    </kuka_lwr_arm>
+    <!-- AluPlate -->
+    <joint name="world_joint2" type="fixed">
+        <origin rpy="0 0 0" xyz="0.0 0.0 0.03"/>
+        <parent link="world"/>
+        <child link="aluplate"/>
+    </joint>
+    <link name="aluplate">
+        <visual>
+            <origin xyz="0 0 0.01"/>
+            <geometry>
+                <box size="0.2 0.2 0.02" xyz="0.0 0.0 0.0"/>
+            </geometry>
+            <material name="Silver"/>
+        </visual>
+        <collision name="aluplate_collision">
+            <geometry>
+                <box size="0.2 0.2 0.02" xyz="0.0 0.0 0.0"/>
+            </geometry>
+        </collision>
+    </link>
+    <gazebo reference="aluplate">
+        <material value="Gazebo/Grey"/>
+    </gazebo>
+    <link name="world"/>
+    <!-- Hand -->
+    <xacro:ahand left="-1" parent_link="lwr_arm_7_link" prefix="ahand" rpy="0 0 0" xyz="0 0 0.1"/>
 </robot>

Commit message: added fixedd link at the center of hand for grasping

File: allegro_kuka_description/models/allegro_hand_on_kuka.urdf.xacro (robot description, xacro)
@@ -63,3 +63,9 @@
     <!-- Hand -->
     <xacro:ahand left="-1" parent_link="lwr_arm_7_link" prefix="ahand" rpy="0 0 0" xyz="0 0 0.1"/>
+    <link name="lwr_exploration_ee"/>
+    <joint name="lwr_exploration_ee_joint" type="fixed">
+        <origin rpy="0 0 0" xyz="0.04 0.0 0.09"/>
+        <parent link="lwr_arm_7_link"/>
+        <child link="lwr_exploration_ee"/>
+    </joint>
 </robot>

Commit message: added joystick control of limbs. and models for pf and without pf

File: allegro_kuka_description/models/allegro_hand_on_kuka.urdf.xacro (robot description, xacro)
@@ -1,71 +1,78 @@
 <robot name="LWR" xmlns:xacro="http://www.ros.org/wiki/xacro">
-    <!-- Some macros used by the urdf -->
-    <xacro:include filename="$(find lwr_description)/model/kuka_lwr_arm.urdf.xacro"/>
-    <xacro:include filename="$(find lwr_description)/model/materials.xml"/>
-    <xacro:include filename="$(find allegro_hand_description_nico)/models/common.urdf.xacro"/>
-    <xacro:include filename="$(find allegro_hand_description_nico)/models/hand.urdf.xacro"/>
-    <!-- This plugin outputs the robot's joint positions and inputs joint torques -->
-    <gazebo>
-        <plugin filename="libmy_robot_plugin.so" name="input_all_torques">
-            <topicName>/lwr/input_torques/ </topicName>
-            <bodyName>lwr_arm_7_link </bodyName>
-        </plugin>
-    </gazebo>
-    <!-- Sets a joint position (for replay)  -->
-    <gazebo>
-        <plugin filename="libset_joint_position_plugin.so" name="set_joint_position">
-            <topicName>/set_gazebo_joint_states </topicName>
-        </plugin>
-    </gazebo>
-    <!-- Streams the contacts  -->
-    <gazebo>
-        <plugin filename="libgazebo_ros_my_contact_plugin.so" name="link_collision_sensor">
-            <always_on>true</always_on>
-            <update_rate>20</update_rate>
-            <bumperTopicName>/link_collision_sensor</bumperTopicName>
-        </plugin>
-    </gazebo>
+<!-- Some macros used by the urdf -->
+<xacro:include filename="$(find lwr_description)/model/kuka_lwr_arm.urdf.xacro"/>
+<xacro:include filename="$(find lwr_description)/model/materials.xml"/>
+<xacro:include filename="$(find allegro_hand_description_nico)/models/common.urdf.xacro"/>
+<xacro:include filename="$(find allegro_hand_description_nico)/models/hand.urdf.xacro"/>
+<!-- This plugin outputs the robot's joint positions and inputs joint torques -->
+<gazebo>
+<plugin filename="libmy_robot_plugin.so" name="input_all_torques">
+<topicName>/lwr/input_torques/ </topicName>
+<bodyName>lwr_arm_7_link </bodyName>
+</plugin>
+</gazebo>
+<!-- Sets a joint position (for replay)  -->
+<gazebo>
+<plugin filename="libset_joint_position_plugin.so" name="set_joint_position">
+<topicName>/set_gazebo_joint_states </topicName>
+</plugin>
+</gazebo>
+<!-- Streams the contacts  -->
+<gazebo>
+<plugin filename="libgazebo_ros_my_contact_plugin.so" name="link_collision_sensor">
+<always_on>true</always_on>
+<update_rate>20</update_rate>
+<bumperTopicName>/link_collision_sensor</bumperTopicName>
+</plugin>
+</gazebo>
 <!--         <gazebo>
-        <plugin filename="libgazebo_ros_my_world_manager_plugin.so" name="world_manager">
-            <always_on>true</always_on>
-            <update_rate>20</update_rate>
-            <bumperTopicName>/link_collision_sensor</bumperTopicName>
-        </plugin>
-    </gazebo> -->
-    <!-- Kuka -->
-    <kuka_lwr_arm name="lwr" parent="aluplate" right="1" tool_name="">
-        <origin rpy="0 0 0" xyz="0 0 0"/>
-    </kuka_lwr_arm>
-    <!-- AluPlate -->
-    <joint name="world_joint2" type="fixed">
-        <origin rpy="0 0 0" xyz="0.0 0.0 0.03"/>
-        <parent link="world"/>
-        <child link="aluplate"/>
-    </joint>
-    <link name="aluplate">
-        <visual>
-            <origin xyz="0 0 0.01"/>
-            <geometry>
-                <box size="0.2 0.2 0.02" xyz="0.0 0.0 0.0"/>
-            </geometry>
-            <material name="Silver"/>
-        </visual>
-        <collision name="aluplate_collision">
-            <geometry>
-                <box size="0.2 0.2 0.02" xyz="0.0 0.0 0.0"/>
-            </geometry>
-        </collision>
-    </link>
-    <gazebo reference="aluplate">
-        <material value="Gazebo/Grey"/>
-    </gazebo>
-    <link name="world"/>
-    <!-- Hand -->
-    <xacro:ahand left="-1" parent_link="lwr_arm_7_link" prefix="ahand" rpy="0 0 0" xyz="0 0 0.1"/>
-    <link name="lwr_exploration_ee"/>
-    <joint name="lwr_exploration_ee_joint" type="fixed">
-        <origin rpy="0 0 0" xyz="0.04 0.0 0.09"/>
-        <parent link="lwr_arm_7_link"/>
-        <child link="lwr_exploration_ee"/>
-    </joint>
+<plugin filename="libgazebo_ros_my_world_manager_plugin.so" name="world_manager">
+<always_on>true</always_on>
+<update_rate>20</update_rate>
+<bumperTopicName>/link_collision_sensor</bumperTopicName>
+</plugin>
+</gazebo> -->
+<gazebo>
+<plugin name="mylinkforce2" filename="libgazebo_ros_force2.so">
+<topicName> /spacenav/twist/ </topicName>
+<bodyNames> lwr_arm_7_link ahand/finger_1/dof0_link</bodyNames>
+<!-- <bodyNames>  </bodyNames> -->
+</plugin>
+</gazebo>
+<!-- Kuka -->
+<kuka_lwr_arm name="lwr" parent="aluplate" right="1" tool_name="">
+<origin rpy="0 0 0" xyz="0 0 0"/>
+</kuka_lwr_arm>
+<!-- AluPlate -->
+<joint name="world_joint2" type="fixed">
+<origin rpy="0 0 0" xyz="0.0 0.0 0.03"/>
+<parent link="world"/>
+<child link="aluplate"/>
+</joint>
+<link name="aluplate">
+<visual>
+<origin xyz="0 0 0.01"/>
+<geometry>
+<box size="0.2 0.2 0.02" xyz="0.0 0.0 0.0"/>
+</geometry>
+<material name="Silver"/>
+</visual>
+<collision name="aluplate_collision">
+<geometry>
+<box size="0.2 0.2 0.02" xyz="0.0 0.0 0.0"/>
+</geometry>
+</collision>
+</link>
+<gazebo reference="aluplate">
+<material value="Gazebo/Grey"/>
+</gazebo>
+<link name="world"/>
+<!-- Hand -->
+<xacro:ahand left="-1" parent_link="lwr_arm_7_link" prefix="ahand" rpy="0 0 0" xyz="0 0 0.1"/>
+<link name="lwr_exploration_ee"/>
+<joint name="lwr_exploration_ee_joint" type="fixed">
+<origin rpy="0 0 0" xyz="0.04 0.0 0.09"/>
+<parent link="lwr_arm_7_link"/>
+<child link="lwr_exploration_ee"/>
+</joint>
 </robot>
